File: Blank Project 2.kicad_sch (KiCad schematic)
At the start: 11 parts

Commit message: Added a resistor.
Parts:
- added R6: 500R, symbol Device:R
- gave numbers to parts that had none: 1
Changed lines of the file:
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@@
     (effects (font (size 1.27 1.27)) (justify left bottom))
   )
+  (symbol (lib_id "Device:R") (at 118.11 119.38 0) (unit 1)
+    (in_bom yes) (on_board yes) (fields_autoplaced)
+    (property "Reference" "R6" (id 0) (at 120.65 118.1099 0)
+      (effects (font (size 1.27 1.27)) (justify left))
+    )
+    (property "Value" "500R" (id 1) (at 120.65 120.6499 0)
+      (effects (font (size 1.27 1.27)) (justify left))
+    )
+    (property "Footprint" "" (id 2) (at 116.332 119.38 90)
+      (effects (font (size 1.27 1.27)) hide)
+    )
+    (property "Datasheet" "~" (id 3) (at 118.11 119.38 0)
+      (effects (font (size 1.27 1.27)) hide)
+    )
+    (pin "1")
+    (pin "2")
+  )
   (symbol (lib_id "Device:R") (at 129.54 119.38 0) (unit 1)
     (in_bom yes) (on_board yes) (fields_autoplaced)
@@
   (symbol (lib_id "Device:R") (at 184.15 119.38 0) (unit 1)
     (in_bom yes) (on_board yes) (fields_autoplaced)
-    (property "Reference" "R?" (id 0) (at 186.69 118.1099 0)
+    (property "Reference" "R7" (id 0) (at 186.69 118.1099 0)
       (effects (font (size 1.27 1.27)) (justify left))
     )
@@
       (reference "R5") (unit 1) (value "500R") (footprint "")
     )
+    (path "/820a1725-ba88-476c-85ca-3e2d00dd7287"
+      (reference "R6") (unit 1) (value "500R") (footprint "")
+    )
     (path "/b481de0f-1165-4e12-9844-8dcd4c741a83"
-      (reference "R?") (unit 1) (value "R") (footprint "")
-    )
-  )
+      (reference "R7") (unit 1) (value "R") (footprint "")
+    )
+  )

Commit message: Added capacitor.
Parts:
- added C6: 10u, symbol Device:C
Changed lines of the file:
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@@
+    (pin "2")
+  )
+  (symbol (lib_id "Device:C") (at 118.11 135.89 0) (unit 1)
+    (in_bom yes) (on_board yes) (fields_autoplaced)
+    (property "Reference" "C6" (id 0) (at 121.92 134.6199 0)
+      (effects (font (size 1.27 1.27)) (justify left))
+    )
+    (property "Value" "10u" (id 1) (at 121.92 137.1599 0)
+      (effects (font (size 1.27 1.27)) (justify left))
+    )
+    (property "Footprint" "" (id 2) (at 119.0752 139.7 0)
+      (effects (font (size 1.27 1.27)) hide)
+    )
+    (property "Datasheet" "~" (id 3) (at 118.11 135.89 0)
+      (effects (font (size 1.27 1.27)) hide)
+    )
+    (pin "1")
     (pin "2")
   )
@@
       (reference "C5") (unit 1) (value "50u") (footprint "")
     )
+    (path "/3aa0c9ce-fb78-4c3d-990c-6185a3da4c4f"
+      (reference "C6") (unit 1) (value "10u") (footprint "")
+    )
     (path "/d50c0195-bb23-4c47-b9e0-34e366d968a2"

Commit message: Added R8.
Parts:
- added R8: 500R, symbol Device:R
Changed lines of the file:
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@@
     (effects (font (size 1.27 1.27)) (justify left bottom))
+  )
+  (symbol (lib_id "Device:R") (at 105.41 119.38 0) (unit 1)
+    (in_bom yes) (on_board yes) (fields_autoplaced)
+    (property "Reference" "R8" (id 0) (at 107.95 118.1099 0)
+      (effects (font (size 1.27 1.27)) (justify left))
+    )
+    (property "Value" "500R" (id 1) (at 107.95 120.6499 0)
+      (effects (font (size 1.27 1.27)) (justify left))
+    )
+    (property "Footprint" "" (id 2) (at 103.632 119.38 90)
+      (effects (font (size 1.27 1.27)) hide)
+    )
+    (property "Datasheet" "~" (id 3) (at 105.41 119.38 0)
+      (effects (font (size 1.27 1.27)) hide)
+    )
+    (pin "1")
+    (pin "2")
   )
   (symbol (lib_id "Device:R") (at 118.11 119.38 0) (unit 1)
@@
       (reference "R7") (unit 1) (value "R") (footprint "")
     )
-  )
+    (path "/4e4cf3fa-0e37-4d39-85d1-d5f5751c269f"
+      (reference "R8") (unit 1) (value "500R") (footprint "")
+    )
+  )
